Commit message: target, boundary box, multiple cameras working

File: models/kobuki_hexagons_kinect.urdf.xacro (robot description, xacro)
@@ -34,5 +34,5 @@
 	</visual>
   </link>
-  <gazebo reference="orientation_box1"><material>Gazebo/Blue</material></gazebo>
-  <gazebo reference="orientation_box2"><material>Gazebo/Red</material></gazebo>
+  <gazebo reference="orientation_box1"><material>Gazebo/Red</material></gazebo>
+  <gazebo reference="orientation_box2"><material>Gazebo/Orange</material></gazebo>
 </robot>
